File: led board/led board.kicad_sch (KiCad schematic)
At the start: 0 parts

Commit message: 4 commit
Parts:
- added D1, D2, D3, D4: LED, LED_SMD:LED_0805_2012Metric_Pad1.15x1.40mm_HandSolder, symbol Device:LED
- added J1: gnd, Connector_PinHeader_2.54mm:PinHeader_1x02_P2.54mm_Vertical, symbol Connector:Conn_01x02_Pin
- added J2: +5V, Connector_PinHeader_2.54mm:PinHeader_1x02_P2.54mm_Vertical, symbol Connector:Conn_01x02_Pin
- added R1, R2, R3, R4: 1k, Resistor_SMD:R_0805_2012Metric_Pad1.20x1.40mm_HandSolder, symbol Device:R_US
Connections:
- new net: D3.1 (K), D4.1 (K), J1.2 (Pin_2)
- new net: D4.2 (A), R4.1
- new net: D2.2 (A), R2.1
- new net: J2.2 (Pin_2), R1.2, R2.2
- new net: D1.2 (A), R1.1
- new net: D1.1 (K), D2.1 (K), J1.1 (Pin_1)
- new net: D3.2 (A), R3.1
- new net: J2.1 (Pin_1), R3.2, R4.2
