File: Arduino Uno SMD/Arduino Uno SMD.kicad_pcb (KiCad board)
At the start: 2 copper layers, 68.6 x 53.3 mm, 56 parts, among them J1 M20-9980345, J2 M20-9980245, J3 M20-9980345, J4 PPTC101LFBN-RC, J5 PPTC081LFBN-RC, J6 PPTC061LFBN-RC, J7 PPTC081LFBN-RC, J8 USB_C_Receptacle_USB2.0_16P, J9 PJ-102AH, Q1 FDN340P, U1 NCP1117-5.0_SOT223, U2 LP2985-3.3, U3 ATMEGA16U2-MU, U4 ATMEGA328P-MU, U5 LMV358IDGKR, Y1 CSTNE16M0V530000R0, Y2 LFXTAL003240BULK

Commit message: 5 commit
Parts:
- added REF**: ESD-Logo_6.6x6mm_SilkScreen, Symbol:ESD-Logo_6.6x6mm_SilkScreen, F.Cu at (169.9, 104.4)

Commit message: 11 commit
Other:
- board text removed: "GITHUB.COM/SABOGALC"
- board text removed: "SMD"
Changed lines of the file:
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@@
-		)
-	)
-	(gr_text "GITHUB.COM/SABOGALC"
-		(at 180.467 121.539 90)
-		(layer "F.SilkS")
-		(effects
-			(font
-				(size 0.75 0.75)
-				(thickness 0.15)
-				(bold yes)
-			)
-			(justify left bottom)
 		)
 	)
@@
 				(thickness 0.2)
 				(bold yes)
-			)
-			(justify left bottom)
-		)
-	)
-	(gr_text "SMD"
-		(at 166.78 91.64 0)
-		(layer "F.SilkS")
-		(effects
-			(font
-				(size 1 1)
-				(thickness 0.2)
-				(bold yes)
